File: Cape_Beaglebone.sch (KiCad schematic (older format))
At the start: 96 parts, among them P8 BeagleBone_Black_Header, P9 BeagleBone_Black_Header

Commit message: 15_07_18
Parts:
- removed C?: C, symbol C
- removed C? (x4): 0.1u, symbol C
- removed C? (x4): 10u, symbol C
- removed IC? (x4): AD7790BRMZ, SOP50P490X110-10N, symbol AD7790BRMZ
- removed J? (x4): Conn_01x06, symbol Conn_01x06
- removed J? (x2): Conn_01x16, symbol Conn_01x16
- removed L?: I, symbol INDUCTOR
- removed NT?: Net-Tie_2, symbol Net-Tie_2
- removed P? (x9): GNDA3_3, symbol GNDA3_3
- added C10, C11, C12, C9: C, Capacitors_SMD:C_0805, symbol C
- added IC5, IC6: AD7793BRUZ, AD7793BRUZ:SOP65P640X120-16N, symbol AD7793BRUZ
- added J10, J6: Conn_01x12, Connectors_JST:JST_GH_BM12B-GHS-TBT_12x1.25mm_Straight, symbol Conn_01x12
- added J11, J12, J8, J9: Conn_01x08, Connectors_JST:JST_GH_BM08B-GHS-TBT_08x1.25mm_Straight, symbol Conn_01x08
- BAT1: renamed from BAT?; footprint S8411-45R -> S8411-45R:S8411-45R
- C1, C13, C14, C15, C16, C17, C18, C19, C2, C20, C21, C22, C23, C24, C25, C26, C27, C28, C29, C3, C4, C5, C6, C7, C8: renamed from C?; footprint (none) -> Capacitors_SMD:C_0805
- IC1: renamed from IC?; footprint QFN40P300X300X105-25N-D -> MPU-9250:QFN40P300X300X105-25N-D
- IC10: renamed from IC?; footprint SOP50P640X120-38N -> ADS8688IDBT:SOP50P640X120-38N
- IC2, IC3: renamed from IC?; footprint SOIC127P600X160-16N -> HX711:SOIC127P600X160-16N
- IC4: renamed from IC?; footprint SOIC127P800X203-8N -> CAT24C256WI-GT3:SOIC127P800X203-8N
- IC7: renamed from IC?; footprint QFN40P300X300X95-25N-D -> MPU-6500:QFN40P300X300X95-25N-D
- IC8: renamed from IC?; footprint 16-PIN-LPCC -> HMC5883L-TR:16-PIN-LPCC
- IC9: renamed from IC?; footprint BMP180 -> BMP180:BMP180
- J1, J3, J4, J7: renamed from J?; footprint (none) -> Connectors_JST:JST_GH_BM04B-GHS-TBT_04x1.25mm_Straight
- J2: renamed from J?; footprint (none) -> Connectors_JST:JST_GH_BM02B-GHS-TBT_02x1.25mm_Straight
- R1, R10, R11, R12, R13, R14, R2, R3, R4, R5, R6, R7, R8, R9: renamed from R?; footprint (none) -> Resistors_SMD:R_0805
- U1: renamed from U?; footprint SOIC127P1032X265-16N -> DS3231S#:SOIC127P1032X265-16N
- U2: renamed from U?; footprint 4525DO-DS...P -> 4525DO-DS5AI001DP:4525DO-DS...P
- U3: renamed from U?; footprint LGA-16 -> LSM303DLHC:LGA14-3X5X1-14L
- U4: renamed from U?; footprint LGA-16 -> L3GD20TR:L3GD20TR
- gave numbers to parts that had none: 7
Connections:
- net labels added: AIN_10N, AIN_10P, AIN_11N, AIN_11P, AIN_12N, AIN_12P, AIN_13N, AIN_13P, AIN_8N, AIN_8P, AIN_9N, AIN_9P, GND
- net labels removed: +3.3VA, SPI_CS_S6, SPI_CS_S7
- wire segments 502 -> 436
- no-connect marks 37 -> 43
Other:
- note removed: "ESSES DOIS SENSORES PODEM COMUNICAR I2C\nApagar essa nota\n"
- moved on the sheet: C15, C17, C18, C19, U3

Commit message: mfsb_29_07_18
Primeira tentativa do layout
Parts:
- removed BAT1: S8411-45R, S8411-45R:S8411-45R, symbol S8411-45R
- added C21, C26: 1u, Capacitors_SMD:C_0805, symbol C
- added C24: 22u, Capacitors_SMD:C_0805, symbol C
- added C25: 10u, Capacitors_SMD:C_0805, symbol C
- added R13, R14: R, Resistors_SMD:R_0805, symbol R
- renumbered C21 to C22, C22 to C23, C23 to C27, C24 to C28, C25 to C29, C26 to C30, C27 to C31, C28 to C32, C29 to C33, J11 to J10, J12 to J11, J10 to J12, J3 to J2, J4 to J3, J2 to J4, P9 to P1, P8 to P2, R13 to R15, R14 to R16
Connections:
- net labels added: INTERUP_SEN_3
- net labels removed: +BATT, -BATT, INTERUP_SEN_5
- wire segments 436 -> 460
- no-connect marks 43 -> 99
Other:
- moved on the sheet: C13, C14, J4, U1

Commit message: Revisões no esquemático do RTC.
Parts:
- removed SW1: Push, symbol SW_Push_Dual_x2
Connections:
- net labels added: INTERUP_RTC
- wire segments 460 -> 459
- no-connect marks 99 -> 98
Other:
- note added: "BBB_P8"
- note added: "BBB_P9"
- moved on the sheet: J4, U1
Changed lines of the file:
@@
 L DS3231S# U1
 U 1 1 5AEBAE29
-P 3400 9350
-F 0 "U1" H 4650 9650 50  0000 L CNN
-F 1 "DS3231S#" H 4650 9550 50  0000 L CNN
-F 2 "DS3231S#:SOIC127P1032X265-16N" H 4650 9450 50  0001 L CNN
-F 3 "https://datasheets.maximintegrated.com/en/ds/DS3231.pdf" H 4650 9350 50  0001 L CNN
-F 4 "Real Time Clock Serial Maxim DS3231S#, Real Time Clock Serial-I2C, 16-Pin SOIC" H 4650 9250 50  0001 L CNN "Description"
-F 5 "2.65" H 4650 9150 50  0001 L CNN "Height"
-F 6 "Maxim Integrated" H 4650 9050 50  0001 L CNN "Manufacturer_Name"
-F 7 "DS3231S#" H 4650 8950 50  0001 L CNN "Manufacturer_Part_Number"
-F 8 "1039915" H 4650 8850 50  0001 L CNN "RS Part Number"
-F 9 "http://uk.rs-online.com/web/p/products/1039915" H 4650 8750 50  0001 L CNN "RS Price/Stock"
-	1    3400 9350
+P 3700 9200
+F 0 "U1" H 4950 9500 50  0000 L CNN
+F 1 "DS3231S#" H 4950 9400 50  0000 L CNN
+F 2 "DS3231S#:SOIC127P1032X265-16N" H 4950 9300 50  0001 L CNN
+F 3 "https://datasheets.maximintegrated.com/en/ds/DS3231.pdf" H 4950 9200 50  0001 L CNN
+F 4 "Real Time Clock Serial Maxim DS3231S#, Real Time Clock Serial-I2C, 16-Pin SOIC" H 4950 9100 50  0001 L CNN "Description"
+F 5 "2.65" H 4950 9000 50  0001 L CNN "Height"
+F 6 "Maxim Integrated" H 4950 8900 50  0001 L CNN "Manufacturer_Name"
+F 7 "DS3231S#" H 4950 8800 50  0001 L CNN "Manufacturer_Part_Number"
+F 8 "1039915" H 4950 8700 50  0001 L CNN "RS Part Number"
+F 9 "http://uk.rs-online.com/web/p/products/1039915" H 4950 8600 50  0001 L CNN "RS Price/Stock"
+	1    3700 9200
 	1    0    0    -1
 $EndComp
@@
 L GNDD #PWR044
 U 1 1 5AEBAE7B
-P 4100 10250
-F 0 "#PWR044" H 4100 10000 50  0001 C CNN
-F 1 "GNDD" H 4100 10125 50  0000 C CNN
-F 2 "" H 4100 10250 50  0001 C CNN
-F 3 "" H 4100 10250 50  0001 C CNN
-	1    4100 10250
+P 4400 10100
+F 0 "#PWR044" H 4400 9850 50  0001 C CNN
+F 1 "GNDD" H 4400 9975 50  0000 C CNN
+F 2 "" H 4400 10100 50  0001 C CNN
+F 3 "" H 4400 10100 50  0001 C CNN
+	1    4400 10100
 	1    0    0    -1
 $EndComp
 $Comp
-L SW_Push_Dual_x2 SW1
-U 1 1 5AEBAE81
-P 3200 9900
-F 0 "SW1" H 3250 10000 50  0000 L CNN
-F 1 "Push" H 3350 10100 50  0000 C CNN
-F 2 "" H 3200 10100 50  0001 C CNN
-F 3 "" H 3200 10100 50  0001 C CNN
-	1    3200 9900
-	0    -1   -1   0
-$EndComp
-$Comp
 L +3V3 #PWR045
 U 1 1 5AEBAE88
-P 3300 9450
-F 0 "#PWR045" H 3300 9300 50  0001 C CNN
-F 1 "+3V3" H 3300 9590 50  0000 C CNN
-F 2 "" H 3300 9450 50  0001 C CNN
-F 3 "" H 3300 9450 50  0001 C CNN
-	1    3300 9450
-	0    -1   -1   0
+P 3550 9300
+F 0 "#PWR045" H 3550 9150 50  0001 C CNN
+F 1 "+3V3" H 3550 9440 50  0000 C CNN
+F 2 "" H 3550 9300 50  0001 C CNN
+F 3 "" H 3550 9300 50  0001 C CNN
+	1    3550 9300
+	1    0    0    -1
 $EndComp
 $Comp
 L GNDD #PWR046
 U 1 1 5AEBAE8E
-P 5000 9850
-F 0 "#PWR046" H 5000 9600 50  0001 C CNN
-F 1 "GNDD" H 5000 9725 50  0000 C CNN
-F 2 "" H 5000 9850 50  0001 C CNN
-F 3 "" H 5000 9850 50  0001 C CNN
-	1    5000 9850
+P 5300 9700
+F 0 "#PWR046" H 5300 9450 50  0001 C CNN
+F 1 "GNDD" H 5300 9575 50  0000 C CNN
+F 2 "" H 5300 9700 50  0001 C CNN
+F 3 "" H 5300 9700 50  0001 C CNN
+	1    5300 9700
 	1    0    0    -1
 $EndComp
@@
 Text GLabel 1150 8100 0    60   Input ~ 0
 SDA_I2C_2
-Text GLabel 4950 9350 2    60   Input ~ 0
+Text GLabel 5250 9200 2    60   Input ~ 0
 SCL_I2C_2
-Text GLabel 4950 9450 2    60   Input ~ 0
+Text GLabel 5250 9300 2    60   Input ~ 0
 SDA_I2C_2
 Text GLabel 3450 8500 0    60   Input ~ 0
@@
 L Conn_01x02 J4
 U 1 1 5AEBAF1C
-P 5300 9900
-F 0 "J4" V 5400 9850 50  0000 C CNN
-F 1 "Conn_01x02" V 5300 9500 50  0001 C CNN
-F 2 "Connectors_JST:JST_GH_BM02B-GHS-TBT_02x1.25mm_Straight" H 5300 9900 50  0001 C CNN
-F 3 "" H 5300 9900 50  0001 C CNN
-	1    5300 9900
+P 5600 9750
+F 0 "J4" V 5700 9700 50  0000 C CNN
+F 1 "Conn_01x02" V 5600 9350 50  0001 C CNN
+F 2 "Connectors_JST:JST_GH_BM02B-GHS-TBT_02x1.25mm_Straight" H 5600 9750 50  0001 C CNN
+F 3 "" H 5600 9750 50  0001 C CNN
+	1    5600 9750
 	0    1    1    0
 $EndComp
@@
 	0    -1   -1   0
 $EndComp
-NoConn ~ 3400 9350
-NoConn ~ 3400 9550
+NoConn ~ 3700 9200
 NoConn ~ 1700 8250
 NoConn ~ 1700 10350
@@
 NoConn ~ 1600 3900
 NoConn ~ 1600 3800
-NoConn ~ 1600 3700
 NoConn ~ 1600 4200
 NoConn ~ 1600 4300
@@
 	1800 10400 1800 10350
 Wire Wire Line
-	4950 9350 4800 9350
-Wire Wire Line
-	4950 9450 4800 9450
-Wire Wire Line
-	3400 9750 3400 10250
-Connection ~ 3400 9850
-Connection ~ 3400 9950
-Wire Wire Line
-	4800 10250 4800 9750
-Connection ~ 4800 9950
-Connection ~ 4800 9850
+	5250 9200 5100 9200
 Wire Wire Line
-	3200 10250 4800 10250
-Connection ~ 3400 10050
-Connection ~ 4800 10050
-Connection ~ 4100 10250
+	5250 9300 5100 9300
 Wire Wire Line
-	3200 9700 3200 9650
+	3700 9600 3700 10100
+Connection ~ 3700 9700
+Connection ~ 3700 9800
 Wire Wire Line
-	3200 9650 3400 9650
+	5100 10100 5100 9600
+Connection ~ 5100 9800
+Connection ~ 5100 9700
+Connection ~ 3700 9900
+Connection ~ 5100 9900
+Connection ~ 4400 10100
 Wire Wire Line
-	3200 10100 3200 10250
-Connection ~ 3400 10250
+	3550 9300 3700 9300
 Wire Wire Line
-	3300 9450 3400 9450
+	5100 9500 5500 9500
 Wire Wire Line
-	4800 9650 5200 9650
-Wire Wire Line
-	4800 9550 5300 9550
+	5100 9400 5600 9400
 Wire Wire Line
 	3500 8200 3600 8200
@@
 	1300 8200 1300 8250
 Wire Wire Line
-	5000 9850 5000 9650
-Connection ~ 5000 9650
+	5300 9700 5300 9500
+Connection ~ 5300 9500
 Wire Wire Line
 	9850 7600 9950 7600
@@
 Wire Wire Line
 	4000 4100 4100 4100
-NoConn ~ 4100 3500
 NoConn ~ 4100 3600
 NoConn ~ 4100 3700
 NoConn ~ 4100 3800
-NoConn ~ 4600 3800
 NoConn ~ 4600 3700
 NoConn ~ 4600 3600
@@
 HX2_SCK
 Wire Wire Line
-	5200 9650 5200 9700
+	5500 9500 5500 9550
 Wire Wire Line
-	5300 9550 5300 9700
+	5600 9400 5600 9550
 Wire Wire Line
 	9500 1050 9500 1150
@@
 Wire Wire Line
 	12850 1800 13000 1800
+Wire Wire Line
+	3700 10100 5100 10100
+NoConn ~ 3700 9500
+Text GLabel 3600 9400 0    60   Input ~ 0
+INTERUP_RTC
+Wire Wire Line
+	3600 9400 3700 9400
+Text Notes 4200 2450 0    60   ~ 0
+BBB_P8
+Text Notes 1700 2450 0    60   ~ 0
+BBB_P9
+Text GLabel 1500 3700 0    60   Input ~ 0
+INTERUP_RTC
+NoConn ~ 4100 3500
+Wire Wire Line
+	1600 3700 1500 3700
+NoConn ~ 4600 3800
 $EndSCHEMATC

Commit message: Revisões no esquemático do HX711.
Parts:
- removed J2: Conn_01x04, Connectors_JST:JST_GH_BM04B-GHS-TBT_04x1.25mm_Straight, symbol Conn_01x04
Other:
- moved on the sheet: C2, C3, J1, Q1, R2, R3

Commit message: Revisões no esquemático do AD7793.
Parts:
- removed J12: Conn_01x12, Connectors_JST:JST_GH_BM12B-GHS-TBT_12x1.25mm_Straight, symbol Conn_01x12
- added J? (x2): Conn_01x06, symbol Conn_01x06
Connections:
- net labels added: IOUT_3, IOUT_4
- wire segments 459 -> 461
- no-connect marks 98 -> 96

Commit message: Revisões no esquemático do ADS8688.
Parts:
- removed J10, J11, J8, J9: Conn_01x08, Connectors_JST:JST_GH_BM08B-GHS-TBT_08x1.25mm_Straight, symbol Conn_01x08
- added J? (x8): Conn_01x04, symbol Conn_01x04
Connections:
- wire segments 461 -> 543

Commit message: Layout com SJT GH
Layout quase finalizado usando os conectores SJT GH de 1,25 mm
Parts:
- removed C10, C9: C, Capacitors_SMD:C_0805, symbol C
- removed C17: 22u, Capacitors_SMD:C_0805, symbol C
- removed C18: 4.7u, Capacitors_SMD:C_0805, symbol C
- removed C6: 10u, Capacitors_SMD:C_0805, symbol C
- removed C7: 0.1u, Capacitors_SMD:C_0805, symbol C
- removed IC3: HX711, HX711:SOIC127P600X160-16N, symbol HX711
- removed IC5: AD7793BRUZ, AD7793BRUZ:SOP65P640X120-16N, symbol AD7793BRUZ
- removed J3, J7: Conn_01x04, Connectors_JST:JST_GH_BM04B-GHS-TBT_04x1.25mm_Straight, symbol Conn_01x04
- removed J6: Conn_01x12, Connectors_JST:JST_GH_BM12B-GHS-TBT_12x1.25mm_Straight, symbol Conn_01x12
- removed Q2: BC807, TO_SOT_Packages_SMD:SOT-23, symbol BC807
- removed R5, R6: R, Resistors_SMD:R_0805, symbol R
- removed U3: LSM303D, LSM303DLHC:LGA14-3X5X1-14L, symbol LSM303D
- removed U4: L3GD20, L3GD20TR:L3GD20TR, symbol L3GD20
- added C12, C13: C, Capacitors_SMD:C_0805, symbol device:C
- added C17: 4.7u, Capacitors_SMD:C_0805, symbol device:C
- added C6: 10u, Capacitors_SMD:C_0805, symbol device:C
- added C7: 0.1u, Capacitors_SMD:C_0805, symbol device:C
- added C9: 22u, Capacitors_SMD:C_0805, symbol Device:C_Small
- added IC13: L3GD20H, L3GD20H_CORRETO:LGA(3X3X1.0-16L), symbol L3GD20H_CORRETO:L3GD20H
- added IC4: HX711, HX711:SOIC127P600X160-16N, symbol HX711:HX711
- added IC7: AD7793BRUZ, AD7793BRUZ:SOP65P640X120-16N, symbol AD7793BRUZ:AD7793BRUZ
- added IC9: LSM303D, LSM303D:PQFN50P300X300X100-16N, symbol LSM303D:LSM303D
- added J2: Conn_01x04, Connectors_JST:JST_GH_BM04B-GHS-TBT_04x1.25mm_Straight, symbol conn:Conn_01x04
- added J4, J6: Conn_01x06, Connectors_JST:JST_GH_BM06B-GHS-TBT_06x1.25mm_Straight, symbol conn:Conn_01x06
- added Q2: BC807, TO_SOT_Packages_SMD:SOT-23, symbol transistors:BC807
- added R5, R6: R, Resistors_SMD:R_0603, symbol device:R
- C1: renamed from C2; symbol C -> device:C
- C10: renamed from C11; symbol C -> device:C
- C11: renamed from C12; symbol C -> device:C
- C14: renamed from C13; symbol C -> device:C
- C15: renamed from C14; symbol C -> device:C
- C16, C23, C24, C25, C26, C3, C33, C4, C5, C8: symbol C -> device:C
- C18: renamed from C15; symbol C -> device:C
- C19: renamed from C20; symbol C -> device:C
- C2: renamed from C1; symbol C -> device:C
- C20: renamed from C21; symbol C -> device:C
- C21: renamed from C22; symbol C -> device:C
- C22: renamed from C19; symbol C -> device:C
- C27: renamed from C30; symbol C -> device:C
- C28: renamed from C27; symbol C -> device:C
- C29: renamed from C31; symbol C -> device:C
- C30: renamed from C32; symbol C -> device:C
- C31: renamed from C28; symbol C -> device:C
- C32: renamed from C29; symbol C -> device:C
- IC1: symbol MPU-9250 -> MPU-9250:MPU-9250
- IC10: renamed from IC8; symbol HMC5883L-TR -> HMC5883L-TR:HMC5883L-TR
- IC11: renamed from IC9; symbol BMP180 -> BMP180:BMP180
- IC12: renamed from IC10; symbol ADS8688IDBT -> ADS8688IDBT:ADS8688IDBT
- IC2: symbol HX711 -> HX711:HX711
- IC3: renamed from U1; value DS3231S# -> DS3231S; symbol DS3231S# -> DS3231S#:DS3231S#
- IC5: renamed from IC4; symbol CAT24C256WI-GT3 -> CAT24C256WI-GT3:CAT24C256WI-GT3
- IC6: symbol AD7793BRUZ -> AD7793BRUZ:AD7793BRUZ
- IC8: renamed from IC7; symbol MPU-6500 -> MPU-6500:MPU-6500
- J1: symbol Conn_01x04 -> conn:Conn_01x04
- J10, J12, J13, J14, J15, J7, J8, J9: renamed from J?; footprint (none) -> Connectors_JST:JST_GH_BM04B-GHS-TBT_04x1.25mm_Straight; symbol Conn_01x04 -> conn:Conn_01x04
- J11, J16: renamed from J?; footprint (none) -> Connectors_JST:JST_GH_BM06B-GHS-TBT_06x1.25mm_Straight; symbol Conn_01x06 -> conn:Conn_01x06
- J3: renamed from J4; symbol Conn_01x02 -> conn:Conn_01x02
- J5: footprint (none) -> complemento2:test_pad; symbol TEST_1P -> conn:TEST_1P
- L1: footprint (none) -> Resistors_THT:R_Axial_DIN0204_L3.6mm_D1.6mm_P7.62mm_Horizontal; symbol INDUCTOR -> pspice1:INDUCTOR
- NT1: footprint (none) -> complementos:net_tie2; symbol Net-Tie_2 -> device:Net-Tie_2
- P1, P2: symbol BeagleBone_Black_Header -> Cape_Beaglebone-rescue:BeagleBone_Black_Header
- Q1: symbol BC807 -> transistors:BC807
- R1: renamed from R2; footprint Resistors_SMD:R_0805 -> Resistors_SMD:R_0603; symbol R -> device:R
- R10, R11, R12, R13, R14, R15, R16, R4, R7, R8, R9: footprint Resistors_SMD:R_0805 -> Resistors_SMD:R_0603; symbol R -> device:R
- R2: renamed from R3; footprint Resistors_SMD:R_0805 -> Resistors_SMD:R_0603; symbol R -> device:R
- R3: renamed from R1; footprint Resistors_SMD:R_0805 -> Resistors_SMD:R_0603; symbol R -> device:R
- SW1: renamed from SW2; footprint (none) -> Buttons_Switches_SMD:SW_DIP_x2_W8.61mm_Slide_LowProfile; symbol SW_DIP_x02 -> Switch1:SW_DIP_x02
- U1: renamed from U2; symbol 4525DO-DS5AI001DP -> 4525DO-DS5AI001DP:4525DO-DS5AI001DP
Connections:
- net labels added: IOUT_1, IOUT_2
- net labels removed: +5V, AIN_10N, AIN_10P, AIN_12N, AIN_12P, GND, GNDA_ADC, PWR_BUT, SYS_RESETN, VDD_ADC
- wire segments 543 -> 527
- no-connect marks 96 -> 108
Other:
- moved on the sheet: C18, C22, C28, C31, C32, U1

Commit message: Final V1.0
Primeria versão final sem revisão
Parts:
- added C34: C, Capacitors_SMD:C_0805, symbol device:C
- added L2: I, Resistors_THT:R_Axial_DIN0204_L3.6mm_D1.6mm_P7.62mm_Horizontal, symbol pspice1:INDUCTOR
- added NT2: Net-Tie_2, complementos:net_tie2, symbol device:Net-Tie_2
- added R17, R18: 0, Resistors_SMD:R_0603, symbol device:R
- J1, J10, J12, J13, J14, J15, J2, J7, J8, J9: footprint Connectors_JST:JST_GH_BM04B-GHS-TBT_04x1.25mm_Straight -> Connectors_JST:JST_SH_BM04B-SRSS-TB_04x1.00mm_Straight
- J11, J16, J4, J6: footprint Connectors_JST:JST_GH_BM06B-GHS-TBT_06x1.25mm_Straight -> Connectors_JST:JST_SH_BM06B-SRSS-TB_06x1.00mm_Straight
- J3: footprint Connectors_JST:JST_GH_BM02B-GHS-TBT_02x1.25mm_Straight -> Connectors_JST:JST_SH_BM02B-SRSS-TB_02x1.00mm_Straight
- SW1: footprint Buttons_Switches_SMD:SW_DIP_x2_W8.61mm_Slide_LowProfile -> Buttons_Switches_SMD:SW_DIP_x2_W5.08mm_Slide_Copal_CHS-A
Connections:
- net labels added: +5V, +5VA_aux, GNDA_ADC, GNDA_aux, VDD_ADC
- net labels removed: SYS_5V
- wire segments 527 -> 555
- no-connect marks 108 -> 106
Other:
- moved on the sheet: C1, C6, J11, J16, R7, R8, R9
